Commit message: More hacking: made some cylinders that don't fall over for align-cylinder-in-zone

File: cliport/environments/assets/cylinder/cylinder.urdf (robot description, URDF)
Before this commit: robot cylinder.urdf, 1 links, 0 joints
Links:
- link baseLink: geometry collision cylinder length=0.1 radius=0.02; visual cylinder length=0.1 radius=0.02
